File: sw-radio/CAD/si4732_radio/microcontroller.kicad_sch (KiCad schematic)
At the start: 1 part, among them U2 ESP32_DevKit_V1_DOIT

Commit message: Further incremental changes
Other:
- title: (none) -> FM/AM/SW Radio
- moved on the sheet: U2
Changed lines of the file:
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@@
 	(generator_version "9.0")
 	(paper "A4")
+	(title_block
+		(title "FM/AM/SW Radio")
+		(date "2026-01-10")
+		(rev "0.1")
+	)
 	(symbol
 		(lib_id "esp32_devkit_v1_doit:ESP32_DevKit_V1_DOIT")
-		(at 148.59 92.71 0)
+		(at 138.43 92.71 0)
 		(unit 1)
 		(exclude_from_sim no)
@@
 		(fields_autoplaced yes)
 		(property "Reference" "U2"
-			(at 150.7333 54.61 0)
+			(at 140.5733 54.61 0)
 			(effects
 				(font
@@
 		)
 		(property "Value" "ESP32_DevKit_V1_DOIT"
-			(at 150.7333 57.15 0)
+			(at 140.5733 57.15 0)
 			(effects
 				(font
@@
 		)
 		(property "Footprint" "doit-esp32-devkit:esp32_devkit_v1_doit"
-			(at 137.16 58.42 0)
+			(at 127 58.42 0)
 			(effects
 				(font
@@
 		)
 		(property "Datasheet" ""
-			(at 137.16 58.42 0)
+			(at 127 58.42 0)
 			(effects
 				(font
@@
 		)
 		(property "Description" "32-bit microcontroller module with WiFi and Bluetooth"
-			(at 148.59 92.71 0)
+			(at 138.43 92.71 0)
 			(effects
 				(font

Commit message: Further incremental changes
Connections:
- net TOUCH7: now reaches U2.10 (IO27)
- net TOUCH6: now reaches U2.11 (IO14)
- net TOUCH5: now reaches U2.12 (IO12)
- net TOUCH4: now reaches U2.13 (IO13)
- net GND: now reaches U2.14 (GND)
- net GND: now also U2.17 (GND)
- net VDD_ESP_3V3: now reaches U2.16 (3V3)
- net TOUCH3: now reaches U2.18 (IO15)
- net TXD2: now reaches U2.22 (IO17)
- net RXD2: now reaches U2.24 (IO18)
- net RSTB_RADIO: now reaches U2.25 (IO19)
- net I2C_SDA: now reaches U2.26 (IO21)
- net I2C_SCL: now reaches U2.29 (IO22)
- net TOUCH9: now reaches U2.6 (IO32)
- net TOUCH8: now reaches U2.7 (IO33)
Other:
- company: (none) -> cyberphox
- moved on the sheet: U2
