File: sw-radio/CAD/si4732_radio/radio.kicad_sch (KiCad schematic)
At the start: 14 parts, among them SW1 SW_SPDT, U1 Si4732-A10-GS, Y1 Crystal

Commit message: Further incremental changes
Parts:
- added C7, C8: 4.7uF, symbol Device:C
- added J1: AudioJack3, symbol Connector_Audio:AudioJack3
- added R1: DNF, symbol Device:R
- added R2: 0R, symbol Device:R
Connections:
- net GND: now also J1.S, R2.2
- net at U1.1 (LOUT/[DFS]): now also C8.1
- net SENB: now reaches U1.10 (~{SEN})
- net SENB: now also R1.2, R2.1
- net VDD_RADIO_3V3: now reaches C1.1, U1.14 (VDD)
- net VDD_RADIO_3V3: now also R1.1
- net at U1.16 (ROUT/[DOUT]): now also C7.1
- net RSTB: now reaches U1.9 (~{RST})
- new net: C8.2, J1.T
- new net: C7.2, J1.R
- no-connect marks 2 -> 4
Other:
- note added: "I2C ADDRESS (SI4732) 0x63 SENB=0V 0x11 SENN=VDD"
- title: (none) -> FM/AM/SW Radio

Commit message: Further incremental changes
Parts:
- removed R1: DNF, symbol Device:R
- removed R2: 0R, symbol Device:R
- added C10: 22nF, Capacitor_SMD:C_0402_1005Metric, symbol Device:C
- added C5: 22nF, symbol Device:C
- added JP1: Solder 1:2, Jumper:SolderJumper-3_P2.0mm_Open_TrianglePad1.0x1.5mm, symbol Jumper:SolderJumper_3_Open
- added R10, R11, R9: 0R, Resistor_SMD:R_0402_1005Metric, symbol Device:R
- added R5, R6: 4K7, Resistor_SMD:R_0402_1005Metric, symbol Device:R
- added Y2: TG2520SMN-32.768Mhz-xxxxNM, Oscillator:Oscillator_SMD_SeikoEpson_TG2520SMN-xxx-xxxxxx-4Pin_2.5x2.0mm, symbol Oscillator:TG2520SMN-xx.xxxxxxMhz-xxxxNM
- C8: renamed from C4; value 18pF -> 22pF
- C9: renamed from C6; value 18pF -> 22pF
- Y1: value Crystal -> 32.768KHz
- renumbered C2 to C1, C3 to C2, C5 to C3, C1 to C4, C7 to C6, C8 to C7, L3 to L1, L1 to L3
Connections:
- net GND: now also C10.2, C5.2, JP1.1 (A), Y2.2 (GND)
- net RCLK: now also R10.2, R9.1; no longer C9.2, Y1.2
- net SCL: now also R6.2
- net SDA: now also R5.2
- net SENB: now also JP1.2 (C)
- net VDD_RADIO_3V3: now also C5.1, JP1.3 (B), R11.1, R5.1, R6.1
- new net: C9.2, R10.1, Y1.2
- new net: C10.1, R11.2, Y2.4 (Vcc)
- new net: R9.2, Y2.3 (OUT)
Other:
- note added: "AM Trap Fc_trap = 1/(2*pi*sqrt(C3*L1))"
- note added: "AM only C2 = 0.47uF Z5U/X7R | AC coupling L3 = 180-450uF"
- note added: "FM/WB Whip only C1 = 1nF | AC coupling L2 = 56nH"
- note added: "I2C ADDRESS (SI4732) 0x63 SENB=0V 0x11 SENB=VDD"
- note added: "RCLK range: 31.130MHz 32.768MHz 40.000MHz prescaler = 1 to 4095"
- note removed: "AM Trap Fc_trap = 1/(2*pi*sqrt(C5*L1))"
- note removed: "C3 = 0.47uF Z5U/X7R | AC coupling L1 = 180 -450uF"
- note removed: "FM/WB Whip only C2 = 1nF | AC coupling L2 = 56nH"
- note removed: "I2C ADDRESS (SI4732) 0x63 SENB=0V 0x11 SENN=VDD"
- company: (none) -> cyberphox
- moved on the sheet: C6, C7, C8, C9, J1, Y1
