File: sw-radio/CAD/si4732_radio/si4732_radio.kicad_sch (KiCad schematic)
At the start: 0 parts

Commit message: Further incremental changes
Parts:
- added AE1: Antenna, symbol Device:Antenna
Connections:
- new net radio/ANT: AE1.1 (A)
Other:
- sheet radio ports: added ANT, RSTB; removed none
- title: (none) -> FM/AM/SW Radio
Changed lines of the file:
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@@
 	(generator_version "9.0")
 	(paper "A4")
+	(title_block
+		(title "FM/AM/SW Radio")
+		(date "2026-01-10")
+		(rev "0.1")
+	)
+	(wire
+		(pts
+			(xy 20.32 78.74) (xy 20.32 86.36)
+		)
+		(stroke
+			(width 0)
+			(type default)
+		)
+	)
+	(wire
+		(pts
+			(xy 20.32 86.36) (xy 29.21 86.36)
+		)
+		(stroke
+			(width 0)
+			(type default)
+		)
+	)
 	(image
-		(at 82.55 114.3)
-		(scale 0.571479)
+		(at 73.66 106.68)
+		(scale 0.439424)
 		(data "iVBORw0KGgoAAAANSUhEUgAAA6wAAAJKCAIAAACnM184AAAAA3NCSVQICAjb4U/gAAAACXBIWXMA"
 			"ABcMAAAXDAGKAo5mAAAgAElEQVR4nOzdZ3wUVdsw8Glb03th0yukkEIooRN6FQyoRJCmgIAR1Fs0"
@@
 		)
 	)
+	(symbol
+		(lib_id "Device:Antenna")
+		(at 20.32 73.66 0)
+		(unit 1)
+		(exclude_from_sim no)
+		(in_bom yes)
+		(on_board yes)
+		(dnp no)
+		(fields_autoplaced yes)
+		(property "Reference" "AE1"
+			(at 22.86 73.0249 0)
+			(effects
+				(font
+					(size 1.27 1.27)
+				)
+				(justify left)
+			)
+		)
+		(property "Value" "Antenna"
+			(at 22.86 75.5649 0)
+			(effects
+				(font
+					(size 1.27 1.27)
+				)
+				(justify left)
+			)
+		)
+		(property "Footprint" ""
+			(at 20.32 73.66 0)
+			(effects
+				(font
+					(size 1.27 1.27)
+				)
+				(hide yes)
+			)
+		)
+		(property "Datasheet" "~"
+			(at 20.32 73.66 0)
+			(effects
+				(font
+					(size 1.27 1.27)
+				)
+				(hide yes)
+			)
+		)
+		(property "Description" "Antenna"
+			(at 20.32 73.66 0)
+			(effects
+				(font
+					(size 1.27 1.27)
+				)
+				(hide yes)
+			)
+		)
+		(pin "1"
+		)
+		(instances
+			(project ""
+				(path "/36dd014e-e30b-45c0-a07c-7db6faee7cad"
+					(reference "AE1")
+					(unit 1)
+				)
+			)
+		)
+	)
 	(sheet
 		(at 29.21 81.28)
-		(size 109.22 67.31)
+		(size 86.36 50.8)
 		(exclude_from_sim no)
 		(in_bom yes)
@@
 		)
 		(property "Sheetfile" "radio.kicad_sch"
-			(at 29.21 149.1746 0)
+			(at 29.21 132.6646 0)
 			(effects
 				(font
@@
 		)
 		(pin "SDA" input
-			(at 138.43 88.9 0)
+			(at 115.57 88.9 0)
 			(effects
 				(font
@@
 		)
 		(pin "SCL" bidirectional
-			(at 138.43 86.36 0)
+			(at 115.57 86.36 0)
 			(effects
 				(font
+					(size 1.27 1.27)
+				)
+				(justify right)
+			)
+		)
+		(pin "ANT" bidirectional
+			(at 29.21 86.36 180)
+			(effects
+				(font
+					(size 1.27 1.27)
+				)
+				(justify left)
+			)
+		)
+		(pin "RSTB" bidirectional
+			(at 115.57 93.98 0)
+			(effects
+				(font

Commit message: Further incremental changes
Parts:
- added R1, R2, R3, R4: 0R, symbol Device:R
Connections:
- net radio/RSTB: now also R4.1
- net radio/SCL: now also R1.1
- net radio/SDA: now also R2.1
- new net microcontroller/I2C_SCL: R1.2
- new net microcontroller/I2C_SDA: R2.2
- new net microcontroller/RSTB_RADIO: R4.2
- new net microcontroller/VDD_ESP_3V3: R3.2
- new net radio/VDD_RADIO_3V3: R3.1
Other:
- sheet microcontroller ports: added I2C_SCL, I2C_SDA, RSTB_RADIO, RXD2, TOUCH3, TOUCH4, TOUCH5, TOUCH6, TOUCH7, TOUCH8, TOUCH9, TXD2, VDD_ESP_3V3; removed none
- sheet radio ports: added VDD_RADIO_3V3; removed none
- company: (none) -> cyberphox
