File: sw-radio/CAD/si4732_radio/si4732_radio.kicad_pcb (KiCad board)
At the start: 2 copper layers, 2 parts, among them U1 Si4732-A10-GS, U2 ESP32_DevKit_V1_DOIT

Commit message: Further incremental changes
Parts:
- added D1: RCLAMP0502B, Package_TO_SOT_SMD:SOT-416, F.Cu at (148.8, 58.5)
- added D2: RCLAMP0502B, Package_TO_SOT_SMD:SOT-416, F.Cu at (148.8, 67.0)
- added Y1: Crystal, Crystal:Crystal_SMD_MicroCrystal_CC1V-T1A-2Pin_8.0x3.7mm, F.Cu at (126.3, 74.5)
- moved U2 36.2 mm to (71.0, 54.0)
- moved U1 22.6 mm to (126.6, 61.9)
Connections:
- U1 pad 1: unconnected-(U1-LOUT/[DFS]-Pad1) -> Net-(U1-LOUT/[DFS])
- U1 pad 10: unconnected-(U1-~{SEN}-Pad10) -> /radio/SENB
- U1 pad 11: unconnected-(U1-SCLK-Pad11) -> /radio/i2c_scl
- U1 pad 12: unconnected-(U1-SDIO-Pad12) -> /radio/i2c_sda
- U1 pad 13: unconnected-(U1-RCLK-Pad13) -> /radio/RCLK
- U1 pad 14: unconnected-(U1-VDD-Pad14) -> /radio/VDD_RADIO_3V3
- U1 pad 15: unconnected-(U1-GND-Pad15) -> GND
- U1 pad 16: unconnected-(U1-ROUT/[DOUT]-Pad16) -> Net-(U1-ROUT/[DOUT])
- U1 pad 2: unconnected-(U1-GPO3/[DCLK]-Pad2) -> /radio/GPO3
- U1 pad 6: unconnected-(U1-FMI-Pad6) -> Net-(U1-FMI)
- U1 pad 7: unconnected-(U1-RFGND-Pad7) -> GND
- U1 pad 8: unconnected-(U1-AMI-Pad8) -> Net-(U1-AMI)
- U1 pad 9: unconnected-(U1-~{RST}-Pad9) -> /radio/RSTB

Commit message: Further incremental changes
Parts:
- added C10: 22nF, Capacitor_SMD:C_0402_1005Metric, F.Cu at (126.9, 38.0)
- added JP1: Solder 1:2, Jumper:SolderJumper-3_P2.0mm_Open_TrianglePad1.0x1.5mm, F.Cu at (129.0, 35.0)
- added R10: 0R, Resistor_SMD:R_0402_1005Metric, F.Cu at (124.0, 40.2)
- added R11: 0R, Resistor_SMD:R_0402_1005Metric, F.Cu at (124.0, 42.2)
- added R5: 4K7, Resistor_SMD:R_0402_1005Metric, F.Cu at (124.0, 34.2)
- added R6: 4K7, Resistor_SMD:R_0402_1005Metric, F.Cu at (124.0, 36.2)
- added R9: 0R, Resistor_SMD:R_0402_1005Metric, F.Cu at (124.0, 38.2)
- added Y2: TG2520SMN-32.768Mhz-xxxxNM, Oscillator:Oscillator_SMD_SeikoEpson_TG2520SMN-xxx-xxxxxx-4Pin_2.5x2.0mm, F.Cu at (143.7, 80.0)
- Y1: value Crystal -> 32.768KHz
Connections:
- U2 pad 10: unconnected-(U2-IO27-Pad10) -> /microcontroller/TOUCH7
- U2 pad 11: unconnected-(U2-IO14-Pad11) -> /microcontroller/TOUCH6
- U2 pad 12: unconnected-(U2-IO12-Pad12) -> /microcontroller/TOUCH5
- U2 pad 13: unconnected-(U2-IO13-Pad13) -> /microcontroller/TOUCH4
- U2 pad 14: unconnected-(U2-GND-Pad14) -> GND
- U2 pad 16: unconnected-(U2-3V3-Pad16) -> /microcontroller/VDD_ESP_3V3
- U2 pad 17: unconnected-(U2-GND-Pad17) -> GND
- U2 pad 18: unconnected-(U2-IO15-Pad18) -> /microcontroller/TOUCH3
- U2 pad 22: unconnected-(U2-IO17-Pad22) -> /microcontroller/TXD2
- U2 pad 24: unconnected-(U2-IO18-Pad24) -> /microcontroller/RXD2
- U2 pad 25: unconnected-(U2-IO19-Pad25) -> /microcontroller/RSTB_RADIO
- U2 pad 26: unconnected-(U2-IO21-Pad26) -> /microcontroller/I2C_SDA
- U2 pad 29: unconnected-(U2-IO22-Pad29) -> /microcontroller/I2C_SCL
- U2 pad 6: unconnected-(U2-IO32-Pad6) -> /microcontroller/TOUCH9
- U2 pad 7: unconnected-(U2-IO33-Pad7) -> /microcontroller/TOUCH8
- Y1 pad 2: /radio/RCLK -> Net-(C9-Pad2)
